File: Hacktues-test.kicad_pcb (KiCad board)
At the start: 2 copper layers, 55 x 53 mm, 8 parts, among them J1 INPUT, U1 ESP-32-WROOM, U2 L7805

Commit message: Found&Fixed-Error
Routing:
- net GND: track 106.2 -> 89.6 mm, vias 4 -> 0
- net VDC: track 27.5 -> 38.4 mm, vias 0 -> 2
- net Net-(U1-D33): track 32.0 -> 40.7 mm, vias 0 -> 2
- net VCC: track 48.7 -> 54.3 mm, vias 0 -> 3
- net Net-(D1-K): track 8.20 -> 7.00 mm
- removed copper zone on B.Cu, net GND
- removed copper zone on F.Cu, net GND

Commit message: HardwareV1.1-Fixed
Routing:
- added copper zone on B.Cu, net GND
- added copper zone on F.Cu, net GND
Changed lines of the file:
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@@
+	)
+	(zone
+		(net 1)
+		(net_name "GND")
+		(layers "F.Cu" "B.Cu")
+		(hatch edge 0.5)
+		(connect_pads
+			(clearance 1)
+		)
+		(min_thickness 1)
+		(filled_areas_thickness no)
+		(fill yes
+			(thermal_gap 1)
+			(thermal_bridge_width 1)
+		)
+		(polygon
+			(pts
+				(xy 105 76) (xy 162 76) (xy 162 131) (xy 106 131)
+			)
+		)
 	)
 	(zone
